Commit message: Update robot_core_3.xacro

File: urdf/robot_core_3.xacro (robot description, xacro)
@@ -59,4 +59,5 @@
                 <cylinder length="0.04" radius="0.05"/>
             </geometry>
+            <material name="blue"/>
         <collision>
         <xacro:inertial_cylinder mass="0.1" length="0.05" radius="0.05">

Commit message: Update robot_core_3.xacro

File: urdf/robot_core_3.xacro (robot description, xacro)
@@ -36,8 +36,8 @@
                 <box size="0.3 0.3 0.15"/>
             </geometry>
-        <collision>
+        </collision>
         <xacro:inertial_box mass="0.5" x="0.3" y="0.3" z="0.15">
             <origin xyz="0.15 0 0.075" rpy="0 0 0"/>
-        <xacro:inertial_box>
+        </xacro:inertial_box>
     </link>
     <joint name="left_wheel_joint" type="continuous">
@@ -60,8 +60,8 @@
             </geometry>
             <material name="blue"/>
-        <collision>
+        </collision>
         <xacro:inertial_cylinder mass="0.1" length="0.05" radius="0.05">
             <origin xyz="0 0 0" rpy="0 0 0"/>
-        <xacro:inertial_cylinder>
+        </xacro:inertial_cylinder>
         <!--                    ^^^추가^^^                     -->
     </link>
