Commit message: Update robot_core_2.xacro

File: urdf/robot_core_2.xacro (robot description, xacro)
@@ -37,8 +37,8 @@
                 <box size="0.3 0.3 0.15"/>
             </geometry>
-        <collision>
+        </collision>
         <xacro:inertial_box mass="0.5" x="0.3" y="0.3" z="0.15">
             <origin xyz="0.15 0 0.075" rpy="0 0 0"/>
-        <xacro:inertial_box>
+        </xacro:inertial_box>
         <!-- ^^^추가^^^ -->
     </link>
